File: hardware/kicad/ESP32_SensorScope/UART.kicad_sch (KiCad schematic)
At the start: 18 parts, among them U6 SN74LV1T125DBV, U7 74LVC1G240DBVRG4, U8 74LVC1G240DBVRG4

Commit message: updatet schematic
Parts:
- removed C3, C4, C5: 100n, symbol Device:C
- removed C7: 3.3n, symbol Device:C
- removed D3: D_Schottky, symbol Device:D_Schottky
- removed D35: 28VDC, symbol Device:D_TVS
- removed D4: 6V8, symbol Device:D_Zener
- removed R14: 100, symbol Device:R
- removed R15: 10K, symbol Device:R
- removed R17: 510, symbol Device:R
- removed R18: 200K, symbol Device:R
- removed R20, R21, R24, R25: 120, symbol Device:R
- removed U6: SN74LV1T125DBV, Package_TO_SOT_SMD:SOT-23-5, symbol Logic_LevelTranslator:SN74LV1T125DBV
- removed U7, U8: 74LVC1G240DBVRG4, Package_TO_SOT_SMD:SOT-23-5, symbol SN74LVC1G240:74LVC1G240DBVRG4
- added C25: 100n, symbol Device:C
- added D20, D21, D22, D26, D27, D28: D_Schottky, symbol Device:D_Schottky
- added D29, D30, D31: 28VDC, symbol Device:D_TVS
- added D32: BAT54S, Package_TO_SOT_SMD:SOT-23, symbol Diode:BAT54S
- added F5, F6: Polyfuse, symbol Device:Polyfuse
- added J17: Conn_01x04_Pin, symbol Connector:Conn_01x04_Pin
- added R45: R, symbol Device:R
- added R68: 220, symbol Device:R
- added R73: 100, symbol Device:R
- added R74: 4K7, symbol Device:R
- added U15, U24: SN74LV1T125DBV, Package_TO_SOT_SMD:SOT-23-5, symbol Logic_LevelTranslator:SN74LV1T125DBV
Connections:
- net +5V: now also C25.1, D20.2 (A), D22.1 (K), D27.1 (K)
- net GND: now also C25.2, D21.2 (A), D26.2 (A), D28.2 (A), D29.1 (A1), D30.1 (A1), D31.1 (A1), J17.4 (Pin_4), U15.3 (GND), U24.3 (GND)
- net UART1_RX: now also U24.4 (Y)
- net UART1_TX: now also U15.2 (A)
- new net: D27.2 (A), D28.1 (K), R68.2, R73.1
- new net: D22.2 (A), D26.1 (K), R74.1, U24.2 (A)
- new net: D20.1 (K), D21.1 (K), D29.2 (A2), F5.1
- new net: F5.2, J17.1 (Pin_1)
- new net: F6.2, J17.2 (Pin_2)
- new net: D31.2 (A2), J17.3 (Pin_3), R74.2
- new net: R68.1, U15.4 (Y)
- new net: D30.2 (A2), F6.1, R73.2
- new net +3.3V: R45.1, U15.5 (VCC), U24.5 (VCC)
- new net UART_nEN: R45.2, U15.1 (~{OE}), U24.1 (~{OE})
Other:
- note removed: "1x Dout"
- note removed: "Invert signal?"

Commit message: addet some footprints"
Parts:
- C25: footprint (none) -> Capacitor_SMD:C_0805_2012Metric
- D20, D21: footprint (none) -> Diode_SMD:D_SMA
Changed lines of the file:
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@@
 			)
 		)
-		(property "Footprint" ""
+		(property "Footprint" "Capacitor_SMD:C_0805_2012Metric"
 			(at 100.0252 67.31 0)
 			(effects
@@
 			)
 		)
-		(property "Footprint" ""
+		(property "Footprint" "Diode_SMD:D_SMA"
 			(at 113.03 63.5 0)
 			(effects
@@
 			)
 		)
-		(property "Footprint" ""
+		(property "Footprint" "Diode_SMD:D_SMA"
 			(at 107.95 59.69 0)
 			(effects
